File: hardware/VK49_2.0.brd (EAGLE design)
At the start: 35 x 35 mm, 65 parts, among them IC1 ATSAMD21G18A-MU, IC2 SPI_FLASH, IC3 MCP73831T-2ACI, IC4 MAX98357AETE+, IC5 DS3231MZ+, IC6 STM6519, IC7 AS1115-BQFT, Q1 LGE2305, Q2 LGE2305, Q3 2N3904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

Commit message: board update
Parts:
- moved JP10 0.41 mm to (10.9, 15.6)
