File: hardware/VK49_2.0.brd (EAGLE design)
At the start: 35 x 35 mm, 65 parts, among them IC1 ATSAMD21G18A-MU, IC2 SPI_FLASH, IC3 MCP73831T-2ACI, IC4 MAX98357AETE+, IC5 DS3231MZ+, IC6 STM6519, IC7 AS1115-BQFT, Q1 LGE2305, Q2 LGE2305, Q3 2N3904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

Commit message: resistor updates
Parts:
- R8: value 30k -> 33k
Changed lines of the file:
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@@
 <attribute name="VENDOR" value="" x="66.548" y="-41.656" size="1.778" layer="27" rot="R90" display="off"/>
 </element>
-<element name="R8" library="BASTL_RESISTORS" library_urn="urn:adsk.eagle:library:32975925" package="RESISTOR0603" package3d_urn="urn:adsk.eagle:package:32975936/2" value="30k" x="29.972" y="25.146" smashed="yes" rot="R90">
+<element name="R8" library="BASTL_RESISTORS" library_urn="urn:adsk.eagle:library:32975925" package="RESISTOR0603" package3d_urn="urn:adsk.eagle:package:32975936/2" value="33k" x="29.972" y="25.146" smashed="yes" rot="R90">
 <attribute name="ASSEMBLED" value="yes" x="75.692" y="-14.478" size="1.778" layer="27" rot="R90" display="off"/>
 <attribute name="MAN" value="" x="75.692" y="-14.478" size="1.778" layer="27" rot="R90" display="off"/>
