File: hardware/VK49_2.0.sch (EAGLE design)
At the start: 60 parts, among them IC1 ATSAMD21G18A-MU, IC2 SPI_FLASH, IC3 MCP73831T-2ACI, IC4 MAX98357AETE+, IC5 DS3231MZ+, IC6 STM6519, J1 USB-C, Q1 LGE2305, Q2 LGE2305, Q3 2N3904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

Commit message: 2.0 board in progress
Parts:
- added C20: 100n, BASTL_CAPACITORS:CAPACITOR0603
- added IC7: AS1115-BQFT, BASTL_ICS:AS1115-BQFT
- added R15, R16: 4k7, BASTL_RESISTORS:RESISTOR0603
- R14: value 100 -> 10k
Connections:
- new net N$12: DISPLAY1.DIG_0, IC7.DIG0
- new net N$13: DISPLAY1.DIG_1, IC7.DIG1
- new net N$14: DISPLAY1.DIG_2, IC7.DIG2
- new net N$15: DISPLAY1.DIG_3, IC7.DIG3
- new net N$16: DISPLAY1.SEG_A, IC7.SEGA
- new net N$17: DISPLAY1.SEG_B, IC7.SEGB
- new net N$18: DISPLAY1.SEG_C, IC7.SEGC
- new net N$19: DISPLAY1.SEG_D, IC7.SEGD
- new net N$20: DISPLAY1.SEG_E, IC7.SEGE
- new net N$21: DISPLAY1.SEG_F, IC7.SEGF
- new net N$22: DISPLAY1.SEG_G, IC7.SEGG
- new net N$23: DISPLAY1.SEG_DP, IC7.SEGDP
- new net N$3: IC7.ISET, R14.1
- net ENABLED: now also R7.1
- net GND: now also C20.1
- net SCL: now also IC7.SCL, R16.1
- net SDA: now also IC7.SDA, R15.1
- net VDD: now also C20.2, IC7.VDD, R14.2, R15.2, R16.2; no longer R7.1
Other:
- moved on the sheet: DISPLAY1, R14

Commit message: 2.0 board routing
Parts:
- removed DISPLAY1: SEG_SR420281N, BASTL_LEDS:SEG_SR420281N
- added DISPLAY: SR420281N, BASTL_LEDS:SEG_SR420281N_NOSILK
- added JP10: VBUS, BASTL_PINHEADERS:M01_ROUND_NO_SILK
- USBC: value USB-C -> TYPE-C-31-M-12
- renumbered J1 to USBC
Connections:
- net ALARM: now also IC1.PA16; no longer IC1.PB08
- net CHRG_STAT: now also IC1.PA18
- net ENABLED: now also IC1.PA17; no longer IC1.PB09
- net GND: now also IC7.EXP, IC7.GND
- net N$12: now also DISPLAY.DIG_0; no longer DISPLAY1.DIG_0
- net N$13: now also DISPLAY.DIG_1; no longer DISPLAY1.DIG_1
- net N$14: now also DISPLAY.DIG_2; no longer DISPLAY1.DIG_2
- net N$15: now also DISPLAY.DIG_3; no longer DISPLAY1.DIG_3
- net N$16: now also DISPLAY.SEG_A; no longer DISPLAY1.SEG_A
- net N$17: now also DISPLAY.SEG_B; no longer DISPLAY1.SEG_B
- net N$18: now also DISPLAY.SEG_C; no longer DISPLAY1.SEG_C
- net N$19: now also DISPLAY.SEG_D; no longer DISPLAY1.SEG_D
- net N$20: now also DISPLAY.SEG_E; no longer DISPLAY1.SEG_E
- net N$21: now also DISPLAY.SEG_F; no longer DISPLAY1.SEG_F
- net N$22: now also DISPLAY.SEG_G; no longer DISPLAY1.SEG_G
- net N$23: now also DISPLAY.SEG_DP; no longer DISPLAY1.SEG_DP
- net VBUS: now also JP10.1

Commit message: resistor updates
Parts:
- R8: value 30k -> 33k
Other:
- note added: "Fully charged (4.2V): 3.158V Discharged (3.2V): 2.406V"
- note removed: "Fully charged (4.2V): 3.231V Discharged (3.2V): 2.462V"
Changed lines of the file:
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@@
 <part name="GND23" library="BASTL_SYMBOLS" library_urn="urn:adsk.eagle:library:32975873" deviceset="GND" device=""/>
 <part name="GND24" library="BASTL_SYMBOLS" library_urn="urn:adsk.eagle:library:32975873" deviceset="GND" device=""/>
-<part name="R8" library="BASTL_RESISTORS" library_urn="urn:adsk.eagle:library:32975925" deviceset="RESISTOR0603" device="" package3d_urn="urn:adsk.eagle:package:32975936/2" value="30k"/>
+<part name="R8" library="BASTL_RESISTORS" library_urn="urn:adsk.eagle:library:32975925" deviceset="RESISTOR0603" device="" package3d_urn="urn:adsk.eagle:package:32975936/2" value="33k"/>
 <part name="R9" library="BASTL_RESISTORS" library_urn="urn:adsk.eagle:library:32975925" deviceset="RESISTOR0603" device="" package3d_urn="urn:adsk.eagle:package:32975936/2" value="100k"/>
 <part name="GND8" library="BASTL_SYMBOLS" library_urn="urn:adsk.eagle:library:32975873" deviceset="GND" device=""/>
@@
 <sheet>
 <plain>
-<text x="38.1" y="-96.52" size="1.778" layer="98">Fully charged (4.2V): 3.231V
-Discharged (3.2V): 2.462V</text>
+<text x="38.1" y="-96.52" size="1.778" layer="98">Fully charged (4.2V): 3.158V
+Discharged (3.2V): 2.406V</text>
 <text x="-238.76" y="111.76" size="12.7" layer="94" ratio="15">VK49 2.0
 Vaclav Mach (vaclavmach@hotmail.cz)
